Commit message: wrist joint functional in gui

File: docker_ws/mia_hand_mujoco/description/ros2_control/mia_hand_mujoco.ros2_control.xacro (robot description, xacro)
@@ -3,5 +3,5 @@
   <xacro:macro
     name="mia_hand_mujoco_ros2_control"
-    params="name prefix xml_model_path hardware_plugin">
+    params="name prefix xml_model_path hardware_plugin include_wrist:=true">
     <ros2_control name="${name}" type="system">
       <hardware>
@@ -26,4 +26,11 @@
       <!-- Extra joints used only for Rviz2 visualization -->
       <joint name="${prefix}j_thumb_opp"/>
+      <xacro:if value="${include_wrist}">
+        <joint name="${prefix}wrist_rotation">
+          <command_interface name="position"/>
+          <state_interface name="position"/>
+          <state_interface name="velocity"/>
+        </joint>
+      </xacro:if>
     </ros2_control>
   </xacro:macro>

File: docker_ws/mia_hand_mujoco/description/urdf/mia_hand_system_interface.urdf.xacro (robot description, xacro)
@@ -6,4 +6,5 @@
   <xacro:arg name="joint_limits_config_file" default="joint_limits_config_default.yaml"/>
   <xacro:arg name="prefix" default=""/>
+  <xacro:arg name="include_wrist" default="true"/>
   <!-- Importing Mia Hand macro -->
   <xacro:include filename="$(find mia_hand_description)/urdf/mia_hand.urdf.xacro"/>
@@ -13,20 +14,48 @@
   <xacro:include filename="$(find mia_hand_mujoco)/description/ros2_control/mia_hand_mujoco.ros2_control.xacro"/>
   <link name="world"/>
-  <xacro:mia_hand
-    laterality="$(arg laterality)"
-    joint_limits_config_file="$(arg joint_limits_config_file)"
-    parent="world"
-    prefix="$(arg prefix)">
-    <xacro:if value="${'right' == '$(arg laterality)'}">
-      <origin xyz="0 0 0.2" rpy="1.57 0 0"/>
-    </xacro:if>
-    <xacro:if value="${'left' == '$(arg laterality)'}">
-      <origin xyz="0 0 0.2" rpy="1.57 3.14 0"/>
-    </xacro:if>
-  </xacro:mia_hand>
+  <!-- Wrist rotation joint: massless link + revolute joint on Z axis -->
+  <xacro:if value="$(arg include_wrist)">
+    <link name="$(arg prefix)wrist_link"/>
+    <joint name="$(arg prefix)wrist_rotation" type="revolute">
+      <parent link="world"/>
+      <child link="$(arg prefix)wrist_link"/>
+      <origin xyz="0 0 0" rpy="0 0 0"/>
+      <axis xyz="0 0 1"/>
+      <limit lower="-3.14159" upper="3.14159" effort="100" velocity="6.28"/>
+    </joint>
+  </xacro:if>
+  <xacro:if value="$(arg include_wrist)">
+    <xacro:mia_hand
+      laterality="$(arg laterality)"
+      joint_limits_config_file="$(arg joint_limits_config_file)"
+      parent="$(arg prefix)wrist_link"
+      prefix="$(arg prefix)">
+      <xacro:if value="${'right' == '$(arg laterality)'}">
+        <origin xyz="0 0 0.2" rpy="1.57 0 0"/>
+      </xacro:if>
+      <xacro:if value="${'left' == '$(arg laterality)'}">
+        <origin xyz="0 0 0.2" rpy="1.57 3.14 0"/>
+      </xacro:if>
+    </xacro:mia_hand>
+  </xacro:if>
+  <xacro:unless value="$(arg include_wrist)">
+    <xacro:mia_hand
+      laterality="$(arg laterality)"
+      joint_limits_config_file="$(arg joint_limits_config_file)"
+      parent="world"
+      prefix="$(arg prefix)">
+      <xacro:if value="${'right' == '$(arg laterality)'}">
+        <origin xyz="0 0 0.2" rpy="1.57 0 0"/>
+      </xacro:if>
+      <xacro:if value="${'left' == '$(arg laterality)'}">
+        <origin xyz="0 0 0.2" rpy="1.57 3.14 0"/>
+      </xacro:if>
+    </xacro:mia_hand>
+  </xacro:unless>
   <xacro:mia_hand_mujoco_ros2_control
     name="MiaHandSim"
     prefix="$(arg prefix)"
     xml_model_path="$(arg xml_model_path)"
-    hardware_plugin="$(arg hardware_plugin)"/>
+    hardware_plugin="$(arg hardware_plugin)"
+    include_wrist="$(arg include_wrist)"/>
 </robot>
