Commit message: fix: add effort state interfaces and fix group_vel_ff_controller type

File: src/mia_hand_ros2_control/description/ros2_control/mia_hand.ros2_control.xacro (robot description, xacro)
@@ -14,6 +14,14 @@
         <hardware>
           <plugin>mock_components/GenericSystem</plugin>
-          <!-- <param name="calculate_dynamics">true</param> -->
         </hardware>
+        <joint name="${prefix}j_thumb_fle">
+          <state_interface name="effort" />
+        </joint>
+        <joint name="${prefix}j_index_fle">
+          <state_interface name="effort" />
+        </joint>
+        <joint name="${prefix}j_mrl_fle">
+          <state_interface name="effort" />
+        </joint>
         <joint name="${prefix}j_thumb_opp">
           <command_interface name="position" />
@@ -32,4 +40,5 @@
         <state_interface name="position" />
         <state_interface name="velocity" />
+        <state_interface name="effort" />
       </joint>
       <joint name="${prefix}j_index_fle">
@@ -38,4 +47,5 @@
         <state_interface name="position" />
         <state_interface name="velocity" />
+        <state_interface name="effort" />
       </joint>
       <joint name="${prefix}j_mrl_fle">
@@ -44,4 +54,5 @@
         <state_interface name="position" />
         <state_interface name="velocity" />
+        <state_interface name="effort" />
       </joint>
       <!-- Extra joints used only for Rviz2 visualization -->

Commit message: fix: remove duplicate effort declarations in mock block (common block covers all three actuated joints)

File: src/mia_hand_ros2_control/description/ros2_control/mia_hand.ros2_control.xacro (robot description, xacro)
@@ -15,13 +15,4 @@
           <plugin>mock_components/GenericSystem</plugin>
         </hardware>
-        <joint name="${prefix}j_thumb_fle">
-          <state_interface name="effort" />
-        </joint>
-        <joint name="${prefix}j_index_fle">
-          <state_interface name="effort" />
-        </joint>
-        <joint name="${prefix}j_mrl_fle">
-          <state_interface name="effort" />
-        </joint>
         <joint name="${prefix}j_thumb_opp">
           <command_interface name="position" />
